File: kudox-game/pcb/kicad_files/kudox_game.kicad_pcb (KiCad board)
At the start: 2 copper layers, 145.7 x 130.4 mm, 65 parts, among them K0 KEYSW, K1 KEYSW, K11 KEYSW, K12 KEYSW, K13 KEYSW, K14 KEYSW, K15 KEYSW, K2 KEYSW, K20 KEYSW, K21 KEYSW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

Commit message: Add symbol libraries.
Parts:
- moved U1 168.3 mm to (33.5, 77.7)
- moved REF*** 62.6 mm to (140.9, 115.9) (x2)
- moved D15 11.9 mm to (199.4, 87.6), turned to 180 degrees
- turned K15 to 0 degrees
Routing:
- net col0: track 240.1 -> 84.3 mm, vias 3 -> 0
- net RST: track 140.6 -> 0.00 mm
- net GND: track 141.9 -> 13.6 mm
- net col1: track 179.6 -> 74.9 mm, vias 1 -> 0
- net col3: track 122.2 -> 46.5 mm, vias 2 -> 0
- net col2: track 118.6 -> 48.3 mm
- net row2: track 199.0 -> 133.0 mm, vias 6 -> 0
- net row3: track 175.2 -> 115.1 mm, vias 3 -> 0
- net col5: track 173.1 -> 136.0 mm, vias 1 -> 0
- net row1: track 123.8 -> 90.0 mm
- net col4: track 100.8 -> 70.4 mm
- net col6: track 94.3 -> 74.1 mm
- net row4: track 211.1 -> 191.9 mm
- net row0: track 125.4 -> 118.5 mm
