File: kudox/pcb/kicad_files/kudox.sch (KiCad schematic (older format))
At the start: 70 parts, among them K0 KEYSW, K1 KEYSW, K10 KEYSW, K11 KEYSW, K12 KEYSW, K13 KEYSW, K14 KEYSW, K15 KEYSW, K16 KEYSW, K2 KEYSW, K20 KEYSW, K21 KEYSW, K22 KEYSW, K23 KEYSW, K24 KEYSW, K25 KEYSW, K3 KEYSW, K30 KEYSW, K31 KEYSW, K32 KEYSW, K33 KEYSW, K34 KEYSW, K35 KEYSW, K4 KEYSW, K40 KEYSW, K41 KEYSW, K42 KEYSW, K43 KEYSW, K44 KEYSW, K45 KEYSW, K46 KEYSW, K5 KEYSW, U1 ProMicro

Commit message: Add symbol libraries.
Parts:
- D0, D1, D10, D11, D12, D13, D14, D15, D16, D2, D20, D21, D22, D23, D24, D25, D3, D30, D31, D32, D33, D34, D35, D4, D40, D41, D42, D43, D44, D45, D46, D5: symbol D -> kudox:D
- K0, K1, K10, K11, K12, K13, K14, K15, K16, K2, K20, K21, K22, K23, K24, K25, K3, K30, K31, K32, K33, K34, K35, K4, K40, K41, K42, K43, K44, K45, K46, K5: symbol KEYSW -> kudox:KEYSW
- R1, R2: symbol R -> kudox:R
- RGB_STRIP1: symbol Conn_01x03 -> kudox:Conn_01x03
- RST_SW1: symbol SW_PUSH -> kudox:SW_PUSH
- TRRS1: symbol Audio-Jack-4 -> kudox:Audio-Jack-4
- U1: symbol ProMicro -> kudox:ProMicro
